File: eagle/breakout_SX1278_green.brd (EAGLE design)
At the start: 28.6 x 28.6 mm, 20 parts, among them X1 734120110

Commit message: Added SX1278 outline as an orientation marker
Routing:
- net 3.3V: track 17.1 -> 19.3 mm
- net DIO5: track 30.4 -> 31.4 mm
Other:
- board text added: "SX1278"
Changed lines of the file:
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@@
 <?xml version="1.0" encoding="utf-8"?>
 <!DOCTYPE eagle SYSTEM "eagle.dtd">
-<eagle version="8.0.2">
+<eagle version="8.1.0">
 <drawing>
 <settings>
@@
 <wire x1="2.2225" y1="28.575" x2="0" y2="26.3525" width="0.254" layer="20"/>
 <text x="24.257" y="8.89" size="0.6096" layer="25">GND</text>
-<wire x1="7.493" y1="22.225" x2="21.209" y2="22.225" width="0.254" layer="21"/>
-<wire x1="21.209" y1="22.225" x2="21.209" y2="6.223" width="0.254" layer="21"/>
-<wire x1="21.209" y1="6.223" x2="7.493" y2="6.223" width="0.254" layer="21"/>
-<wire x1="7.493" y1="6.223" x2="7.493" y2="22.225" width="0.254" layer="21"/>
+<wire x1="6.35" y1="22.225" x2="22.352" y2="22.225" width="0.254" layer="21"/>
+<wire x1="22.352" y1="22.225" x2="22.352" y2="6.223" width="0.254" layer="21"/>
+<wire x1="22.352" y1="6.223" x2="6.35" y2="6.223" width="0.254" layer="21"/>
+<wire x1="6.35" y1="6.223" x2="6.35" y2="22.225" width="0.254" layer="21"/>
 <text x="4.445" y="21.717" size="0.6096" layer="25" rot="R180">GND</text>
+<wire x1="13.081" y1="9.144" x2="19.05" y2="9.144" width="0.254" layer="21"/>
+<wire x1="19.05" y1="9.144" x2="19.05" y2="15.113" width="0.254" layer="21"/>
+<wire x1="19.05" y1="15.113" x2="13.081" y2="15.113" width="0.254" layer="21"/>
+<wire x1="13.081" y1="15.113" x2="13.081" y2="9.144" width="0.254" layer="21"/>
+<circle x="13.843" y="14.351" radius="0.127" width="0.254" layer="21"/>
+<text x="14.097" y="13.081" size="0.6096" layer="25">SX1278</text>
 </plain>
 <attributes>
@@
 <wire x1="15.621" y1="25.654" x2="15.621" y2="12.192" width="0.254" layer="16"/>
 <wire x1="15.621" y1="12.192" x2="16.637" y2="11.176" width="0.254" layer="16"/>
-<wire x1="16.637" y1="11.176" x2="19.558" y2="11.176" width="0.254" layer="16"/>
-<via x="19.558" y="11.176" extent="1-16" drill="0.6"/>
-<wire x1="19.558" y1="11.176" x2="22.606" y2="11.176" width="0.254" layer="1"/>
+<wire x1="16.637" y1="11.176" x2="18.161" y2="11.176" width="0.254" layer="16"/>
+<via x="18.161" y="11.176" extent="1-16" drill="0.6"/>
+<wire x1="18.161" y1="11.176" x2="22.606" y2="11.176" width="0.254" layer="1"/>
 </signal>
 <signal name="DIO4">
 <contactref element="JP1" pad="6"/>
 <contactref element="DIO4" pad="1"/>
-<wire x1="22.606" y1="13.208" x2="19.558" y2="13.208" width="0.254" layer="1"/>
-<via x="19.558" y="13.208" extent="1-16" drill="0.6"/>
-<wire x1="19.558" y1="13.208" x2="18.669" y2="13.208" width="0.254" layer="16"/>
-<wire x1="18.669" y1="13.208" x2="18.161" y2="13.716" width="0.254" layer="16"/>
-<wire x1="18.161" y1="13.716" x2="18.161" y2="25.654" width="0.254" layer="16"/>
+<wire x1="22.606" y1="13.208" x2="18.161" y2="13.208" width="0.254" layer="1"/>
+<via x="18.161" y="13.208" extent="1-16" drill="0.6"/>
+<wire x1="18.161" y1="13.208" x2="18.161" y2="25.654" width="0.254" layer="16"/>
 </signal>
 <signal name="DIO5">
 <contactref element="JP1" pad="7"/>
 <contactref element="DIO5" pad="1"/>
-<wire x1="20.701" y1="25.654" x2="20.701" y2="10.414" width="0.254" layer="16"/>
-<wire x1="20.701" y1="10.414" x2="19.431" y2="9.144" width="0.254" layer="16"/>
-<wire x1="19.431" y1="9.144" x2="15.621" y2="9.144" width="0.254" layer="16"/>
-<via x="15.621" y="9.144" extent="1-16" drill="0.6"/>
-<wire x1="15.621" y1="9.144" x2="6.096" y2="9.144" width="0.254" layer="1"/>
+<wire x1="20.701" y1="25.654" x2="20.701" y2="9.652" width="0.254" layer="16"/>
+<wire x1="20.701" y1="9.652" x2="19.431" y2="8.382" width="0.254" layer="16"/>
+<wire x1="19.431" y1="8.382" x2="14.097" y2="8.382" width="0.254" layer="16"/>
+<via x="14.097" y="8.382" extent="1-16" drill="0.6"/>
+<wire x1="14.097" y1="8.382" x2="9.525" y2="8.382" width="0.254" layer="1"/>
+<wire x1="9.525" y1="8.382" x2="8.763" y2="9.144" width="0.254" layer="1"/>
+<wire x1="8.763" y1="9.144" x2="6.096" y2="9.144" width="0.254" layer="1"/>
 </signal>
 <signal name="3.3V">
 <contactref element="VCC" pad="1"/>
-<wire x1="18.161" y1="7.239" x2="18.161" y2="14.224" width="0.4064" layer="1"/>
-<wire x1="18.161" y1="14.224" x2="19.177" y2="15.24" width="0.4064" layer="1"/>
-<wire x1="19.177" y1="15.24" x2="22.606" y2="15.24" width="0.4064" layer="1"/>
+<wire x1="18.161" y1="7.239" x2="16.637" y2="8.763" width="0.4064" layer="1"/>
+<wire x1="16.637" y1="8.763" x2="16.637" y2="14.224" width="0.4064" layer="1"/>
+<wire x1="16.637" y1="14.224" x2="17.653" y2="15.24" width="0.4064" layer="1"/>
+<wire x1="17.653" y1="15.24" x2="22.606" y2="15.24" width="0.4064" layer="1"/>
 <via x="18.161" y="7.239" extent="1-16" drill="0.6"/>
 <contactref element="JP2A" pad="1"/>
@@
 <signal name="SCK">
 <contactref element="SCK" pad="1"/>
-<via x="13.081" y="13.335" extent="1-16" drill="0.6"/>
-<wire x1="13.081" y1="13.335" x2="13.081" y2="14.351" width="0.254" layer="1"/>
-<wire x1="13.081" y1="14.351" x2="12.192" y2="15.24" width="0.254" layer="1"/>
-<wire x1="12.192" y1="15.24" x2="6.096" y2="15.24" width="0.254" layer="1"/>
+<via x="12.319" y="13.335" extent="1-16" drill="0.6"/>
+<wire x1="12.319" y1="13.335" x2="12.319" y2="14.351" width="0.254" layer="1"/>
+<wire x1="12.319" y1="14.351" x2="11.43" y2="15.24" width="0.254" layer="1"/>
+<wire x1="11.43" y1="15.24" x2="6.096" y2="15.24" width="0.254" layer="1"/>
 <contactref element="JP2A" pad="3"/>
-<wire x1="13.081" y1="13.335" x2="13.081" y2="7.874" width="0.254" layer="16"/>
-<wire x1="13.081" y1="7.874" x2="15.113" y2="5.842" width="0.254" layer="16"/>
-<wire x1="15.113" y1="5.842" x2="15.113" y2="2.794" width="0.254" layer="16"/>
+<wire x1="12.319" y1="13.335" x2="12.319" y2="7.874" width="0.254" layer="16"/>
+<wire x1="12.319" y1="7.874" x2="15.113" y2="5.08" width="0.254" layer="16"/>
+<wire x1="15.113" y1="5.08" x2="15.113" y2="2.794" width="0.254" layer="16"/>
 </signal>
 <signal name="MISO">
